File: RotorflightF7.kicad_pcb (KiCad board)
At the start: 2 copper layers, 50 parts, among them J1 Outputs, J2 RX, J3 LED, J4 UART, J5 USB_C_Receptacle_USB2.0, SW1 SW_Push, U1 STM32F722RETx, U2 USBLC6-2SC6, U3 W25Q32JVZP, U4 BMI270, U5 TPS54202DDC, U6 XC6220B331MR, Y1 8MHz

Commit message: stuff
Parts:
- removed D1: RED, LED_SMD:LED_0603_1608Metric
- removed D2: GRN, LED_SMD:LED_0603_1608Metric
- added C20: 100n, Capacitor_SMD:C_0402_1005Metric, F.Cu at (112.7, 79.4)
- added C21: 100n, Capacitor_SMD:C_0402_1005Metric, F.Cu at (114.5, 77.4)
- added D4: DT1240A-08LP3810, Package_DFN_QFN:UDFN-9_1.0x3.8mm_P0.5mm, F.Cu at (101.9, 64.9)
- added D5: LED_KBRG, LED_SMD:LED_WS2812B-2020_PLCC4_2.0x2.0mm, F.Cu at (102.3, 68.3)
- added J6: C, Connector_JST:JST_GH_BM04B-GHS-TBT_1x04-1MP_P1.25mm_Vertical, F.Cu at (122.2, 63.3)
- added R11: 470, Resistor_SMD:R_0402_1005Metric, F.Cu at (99.6, 67.5)
- added R12: 470, Resistor_SMD:R_0402_1005Metric, F.Cu at (99.6, 66.5)
- added R13: 470, Resistor_SMD:R_0402_1005Metric, F.Cu at (99.6, 65.5)
- added R14: 470, Resistor_SMD:R_0402_1005Metric, F.Cu at (99.6, 64.5)
- added R15: 470, Resistor_SMD:R_0402_1005Metric, F.Cu at (99.6, 63.5)
- added R16: 470, Resistor_SMD:R_0402_1005Metric, F.Cu at (99.6, 62.5)
- added R17: 470, Resistor_SMD:R_0402_1005Metric, F.Cu at (99.6, 61.5)
- added R18: 22, Resistor_SMD:R_0402_1005Metric, F.Cu at (134.1, 37.6)
- added R19: 22, Resistor_SMD:R_0402_1005Metric, F.Cu at (134.1, 39.6)
- added R20: 22, Resistor_SMD:R_0402_1005Metric, F.Cu at (134.1, 41.6)
- added R21: 22, Resistor_SMD:R_0402_1005Metric, F.Cu at (120.2, 78.4)
- added R22: 22, Resistor_SMD:R_0402_1005Metric, F.Cu at (117.7, 78.3)
- added R23: 22, Resistor_SMD:R_0402_1005Metric, F.Cu at (137.0, 35.6)
- added R24: 22, Resistor_SMD:R_0402_1005Metric, F.Cu at (137.0, 37.6)
- added R26: 47, Resistor_SMD:R_0402_1005Metric, F.Cu at (102.9, 70.1)
- added R27: 75, Resistor_SMD:R_0402_1005Metric, F.Cu at (101.3, 70.6)
- added U7: SPL06-001, Package_LGA:Bosch_LGA-8_2x2.5mm_P0.65mm_ClockwisePinNumbering, F.Cu at (114.5, 79.5)
- C1, C10, C11, C12, C13, C15, C16, C18, C19, C2, C3, C4, C5, C6, C7, C8, C9: footprint Capacitor_SMD:C_0603_1608Metric -> Capacitor_SMD:C_0402_1005Metric
- J2: value RX -> A; footprint Connector_JST:JST_SH_BM04B-SRSS-TB_1x04-1MP_P1.00mm_Vertical -> Connector_JST:JST_GH_BM04B-GHS-TBT_1x04-1MP_P1.25mm_Vertical
- J3: footprint Connector_JST:JST_SH_BM03B-SRSS-TB_1x03-1MP_P1.00mm_Vertical -> Connector_JST:JST_GH_BM03B-GHS-TBT_1x03-1MP_P1.25mm_Vertical
- J4: value UART -> B; footprint Connector_JST:JST_SH_BM04B-SRSS-TB_1x04-1MP_P1.00mm_Vertical -> Connector_JST:JST_GH_BM04B-GHS-TBT_1x04-1MP_P1.25mm_Vertical
- R1, R10, R2, R5, R6, R7, R8, R9: footprint Resistor_SMD:R_0603_1608Metric -> Resistor_SMD:R_0402_1005Metric
- R3: value 47 -> 10k; footprint Resistor_SMD:R_0603_1608Metric -> Resistor_SMD:R_0402_1005Metric
- R4: value 75 -> 10k; footprint Resistor_SMD:R_0603_1608Metric -> Resistor_SMD:R_0402_1005Metric
- U3: value W25Q32JVZP -> W25N01G; footprint Package_SON:WSON-8-1EP_6x5mm_P1.27mm_EP3.4x4.3mm -> Package_SON:WSON-8-1EP_8x6mm_P1.27mm_EP3.4x4.3mm
- Y1: footprint Crystal:Crystal_SMD_3225-4Pin_3.2x2.5mm -> Crystal:Crystal_SMD_2012-2Pin_2.0x1.2mm
- moved C2 98.7 mm to (120.2, 70.8)
- moved C1 98.2 mm to (120.2, 67.2), turned to 180 degrees
- moved R6 97.8 mm to (124.9, 78.3), turned to 180 degrees
- moved J4 95.3 mm to (130.4, 82.3), turned to 180 degrees
- moved C12 94.9 mm to (119.3, 76.9), turned to 180 degrees
- moved U2 94.7 mm to (123.8, 72.5), turned to 180 degrees
- moved C11 94.6 mm to (117.4, 76.9)
- moved R2 93.8 mm to (122.6, 78.2)
- moved C19 89.5 mm to (110.5, 83.2), turned to -90 degrees
- moved J2 89.1 mm to (121.0, 82.3), turned to 180 degrees
- moved C8 88.7 mm to (114.2, 75.3), turned to 180 degrees
- moved R5 88.4 mm to (124.9, 67.9), turned to 180 degrees
- moved C17 87.9 mm to (104.0, 83.0), turned to 90 degrees
- moved C6 87.9 mm to (116.7, 61.7), turned to 90 degrees
- moved C5 87.7 mm to (115.7, 61.7), turned to 90 degrees
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Connections:
- J1 pad 1: /Out1 -> Net-(J1-Pin_1)
- J1 pad 15: VBUS -> GND
- J1 pad 16: VBUS -> GND
- J1 pad 2: /Out2 -> Net-(J1-Pin_2)
- J1 pad 3: /Out3 -> Net-(J1-Pin_3)
- J1 pad 4: /Out4 -> Net-(J1-Pin_4)
- J1 pad 5: /Out5 -> Net-(J1-Pin_5)
- J1 pad 6: /Out6 -> Net-(J1-Pin_6)
- J1 pad 7: /Out7 -> Net-(J1-Pin_7)
- J1 pad 8: /Out8 -> VBUS
- J2 pad 1: /UART1_TX -> Net-(J2-Pin_1)
- J2 pad 2: /UART1_RX -> Net-(J2-Pin_2)
- J3 pad 1: /LEDOUT -> Net-(J3-Pin_1)
- J4 pad 1: /UART2_TX -> Net-(J4-Pin_1)
- J4 pad 2: /UART2_RX -> Net-(J4-Pin_2)
- R3 pad 1: GND -> +3V3
- R3 pad 2: Net-(D1-K) -> /BARO_SCL
- R4 pad 1: GND -> +3V3
- R4 pad 2: Net-(D2-K) -> /BARO_SDA
- U1 pad 10: unconnected-(U1-PC2-Pad10) -> /5V_ADC
- U1 pad 11: unconnected-(U1-PC3-Pad11) -> /Vx_Curr
- U1 pad 16: /UART2_TX -> /RPM
- U1 pad 17: /UART2_RX -> /SBUS
- U1 pad 20: /OCS_BMI -> /BMI_NSS
- U1 pad 21: /SPI_SCK -> /BMI_SCK
- U1 pad 22: /SPI_MISO -> /BMI_MISO
- U1 pad 23: /SPI_MOSI -> /BMI_MOSI
- U1 pad 24: unconnected-(U1-PC4-Pad24) -> /ESC_Curr
- U1 pad 25: /Out1 -> /S3
- U1 pad 26: /Out2 -> unconnected-(U1-PB1-Pad26)
- U1 pad 28: /Out7 -> /UART3_TX
- U1 pad 29: /Out8 -> /UART3_RX
- U1 pad 3: unconnected-(U1-PC14-Pad3) -> /LED_GR
- U1 pad 33: unconnected-(U1-PB12-Pad33) -> /FLASH_NSS
- U1 pad 34: unconnected-(U1-PB13-Pad34) -> /FLASH_SCK
- U1 pad 35: unconnected-(U1-PB14-Pad35) -> /FLASH_MISO
- U1 pad 36: unconnected-(U1-PB15-Pad36) -> /FLASH_MOSI
- U1 pad 37: unconnected-(U1-PC6-Pad37) -> /UART6_TX
- U1 pad 38: unconnected-(U1-PC7-Pad38) -> /UART6_RX
- U1 pad 4: unconnected-(U1-PC15-Pad4) -> /LED_RD
- U1 pad 41: /CS_BMI -> /LEDOUT
- U1 pad 42: /CS_FLASH -> unconnected-(U1-PA9-Pad42)
- U1 pad 43: unconnected-(U1-PA10-Pad43) -> /DSM
- U1 pad 46: /LED_0 -> /SWDIO
- U1 pad 49: /INT1_BMI -> /SWCLK
- U1 pad 50: /INT2_BMI -> /BMI_INT
- U1 pad 55: /LEDOUT -> /TAIL
- U1 pad 56: /Out3 -> /S1
- U1 pad 57: /Out4 -> /S2
- U1 pad 58: /UART1_TX -> /ESC
- U1 pad 59: /UART1_RX -> unconnected-(U1-PB7-Pad59)
- U1 pad 61: /Out5 -> /BARO_SCL
- U1 pad 62: /Out6 -> /BARO_SDA
- U1 pad 8: unconnected-(U1-PC0-Pad8) -> /VBAT_ADC
- U1 pad 9: unconnected-(U1-PC1-Pad9) -> /Vx_ADC
- U2 pad 1: /USB_D+ -> /USB_D-
- U2 pad 3: /USB_D- -> /USB_D+
- U2 pad 4: /MCU_D- -> /MCU_D+
- U2 pad 5: +5V -> Net-(D3-A)
- U2 pad 6: /MCU_D+ -> /MCU_D-
- U3 pad 1: /CS_FLASH -> /FLASH_NSS
- U3 pad 2: /SPI_MISO -> /FLASH_MISO
- U3 pad 5: /SPI_MOSI -> /FLASH_MOSI
- U3 pad 6: /SPI_SCK -> /FLASH_SCK
- U3 pad 9: GND -> (no net)
- U4 pad 1: /SPI_MISO -> /BMI_MISO
- U4 pad 10: /OCS_BMI -> unconnected-(U4-OSCB-Pad10)
- U4 pad 12: /CS_BMI -> /BMI_NSS
- U4 pad 13: /SPI_SCK -> /BMI_SCK
- U4 pad 14: /SPI_MOSI -> /BMI_MOSI
- U4 pad 4: /INT1_BMI -> /BMI_INT
- U4 pad 9: /INT2_BMI -> unconnected-(U4-INT2-Pad9)
Routing:
- net +5V: track 0.00 -> 78.7 mm, vias 0 -> 6
- net GND: track 0.00 -> 71.1 mm, vias 0 -> 26
- net +3V3: track 0.00 -> 37.5 mm, vias 0 -> 12
- net /BARO_SDA: track 0.00 -> 21.4 mm, vias 0 -> 2
- net /UART6_TX: track 0.00 -> 19.7 mm, vias 0 -> 2
- net /LED_GR: track 0.00 -> 19.3 mm, vias 0 -> 2
- net /BARO_SCL: track 0.00 -> 18.9 mm, vias 0 -> 2
- net /LED_RD: track 0.00 -> 18.2 mm, vias 0 -> 2
- net /BMI_MOSI: track 0.00 -> 17.9 mm, vias 0 -> 2
- net VBUS: track 0.00 -> 17.8 mm
- net /BMI_NSS: track 0.00 -> 17.2 mm, vias 0 -> 2
- net /UART6_RX: track 0.00 -> 16.7 mm, vias 0 -> 2
- net /BMI_SCK: track 0.00 -> 16.5 mm
- net Net-(J4-Pin_2): track 0.00 -> 15.6 mm, vias 0 -> 2
- net /BMI_MISO: track 0.00 -> 14.9 mm
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- added copper zone on In2.Cu, net +3V3
- added copper zone on F.Cu, net GND
- added copper zone on In1.Cu, net GND
- added copper zone on F.Cu, net VBUS
- added copper zone on In2.Cu, net VBUS
Other:
- board outline added: 45 x 25 mm
- copper layers 2 -> 4

Commit message: yes
Parts:
- removed C21, C6, C7: 100n, Capacitor_SMD:C_0402_1005Metric
- removed D4: DT1240A-08LP3810, Package_DFN_QFN:UDFN-9_1.0x3.8mm_P0.5mm
- removed D5: LED_KBRG, LED_SMD:LED_WS2812B-2020_PLCC4_2.0x2.0mm
- removed J6: C, Connector_JST:JST_GH_BM04B-GHS-TBT_1x04-1MP_P1.25mm_Vertical
- removed R20, R22, R23, R24: 22, Resistor_SMD:R_0402_1005Metric
- removed R26: 47, Resistor_SMD:R_0402_1005Metric
- removed R27: 75, Resistor_SMD:R_0402_1005Metric
- added D1: B5819W_C8598, Diode_SMD:D_SOD-123, F.Cu at (120.5, 42.5)
- added D2: Green, LED_SMD:LED_0603_1608Metric, F.Cu at (117.3, 44.3)
- added U8: SPL06-001, Package_LGA:Bosch_LGA-8_2x2.5mm_P0.65mm_ClockwisePinNumbering, F.Cu at (111.6, 50.1)
- added U9: W25N01G, Package_SON:WSON-8-1EP_8x6mm_P1.27mm_EP3.4x4.3mm, B.Cu at (119.5, 60.2)
- C1: value 30p -> 10u; footprint Capacitor_SMD:C_0402_1005Metric -> Capacitor_SMD:C_0603_1608Metric
- C10, C19: value 4.7u -> 100n; moved to B.Cu
- C11: value 100n -> 1u; moved to B.Cu
- C14: value 10u -> 100n; footprint Capacitor_SMD:C_0603_1608Metric -> Capacitor_SMD:C_0402_1005Metric; moved to B.Cu
- C16: value 100p -> 100n
- C17: value 47u -> 100n; footprint Capacitor_SMD:C_0603_1608Metric -> Capacitor_SMD:C_0402_1005Metric; moved to B.Cu
- C18: value 10u -> 100n; moved to B.Cu
- C2: value 30p -> 100n
- C20: value 100n -> 4.7u; moved to B.Cu
- C3: value 2.2u -> 22u; footprint Capacitor_SMD:C_0402_1005Metric -> Capacitor_SMD:C_0603_1608Metric
- C4: value 100n -> 22u; footprint Capacitor_SMD:C_0402_1005Metric -> Capacitor_SMD:C_0603_1608Metric
- C5: value 1u -> 10u; footprint Capacitor_SMD:C_0402_1005Metric -> Capacitor_SMD:C_0603_1608Metric
- C8: value 100n -> 2.2u; moved to B.Cu
- C9: value 100n -> 10u; footprint Capacitor_SMD:C_0402_1005Metric -> Capacitor_SMD:C_0603_1608Metric
- D3: value B5819W_C8598 -> Red; footprint Diode_SMD:D_SOD-123 -> LED_SMD:LED_0603_1608Metric
- H1, H2, H3, H4: footprint MountingHole:MountingHole_3.2mm_M3 -> MountingHole:MountingHole_2.2mm_M2_Pad_Via
- J1: value Outputs -> USB_C_Receptacle_USB2.0; footprint footprints:8xServo -> Connector_USB:USB_C_Receptacle_HRO_TYPE-C-31-M-12
- J2: value A -> Outputs; footprint Connector_JST:JST_GH_BM04B-GHS-TBT_1x04-1MP_P1.25mm_Vertical -> footprints:7xServo_Vertical
- J3: value LED -> A; footprint Connector_JST:JST_GH_BM03B-GHS-TBT_1x03-1MP_P1.25mm_Vertical -> Connector_JST:JST_GH_BM04B-GHS-TBT_1x04-1MP_P1.25mm_Vertical
- J4: value B -> DSM; footprint Connector_JST:JST_GH_BM04B-GHS-TBT_1x04-1MP_P1.25mm_Vertical -> footprints:JST_ZH_B3B-ZR_1x03_P1.50mm_Vertical
- J5: value USB_C_Receptacle_USB2.0 -> JTAG_TC2030; footprint Connector_USB:USB_C_Receptacle_HRO_TYPE-C-31-M-12 -> marbastlib_various:CON_TC2030_outlined
- L1: value 10uH -> CSME0418D-4R7M-LRH; footprint Inductor_SMD:L_Sunlord_MWSA0402S -> Inductor_SMD:L_Vishay_IFSC-1515AH_4x4x1.8mm
- R1, R2, R3, R4: value 10k -> 470
- R10: value 13.7k -> 10k
- R11, R12, R13: value 470 -> 10k; moved to B.Cu
- R14, R15: value 470 -> 10k
- R16, R17: value 470 -> 22
- R18: value 22 -> 75
- R19: value 22 -> 47
- R5, R6: value 5.1k -> 470
- R7: value 10k -> 22r
- R8: value 10k -> 5.1k
- R9: value 100k -> 5.1k
- U1: value STM32F722RETx -> ESD1014; footprint Package_QFP:LQFP-64_10x10mm_P0.5mm -> Package_DFN_QFN:DFN-10-1EP_2.6x2.6mm_P0.5mm_EP1.3x2.2mm
- U2: value USBLC6-2SC6 -> AP63205WU; footprint Package_TO_SOT_SMD:SOT-23-6 -> Package_TO_SOT_SMD:TSOT-23-6
- U3: value W25N01G -> ESD1014; footprint Package_SON:WSON-8-1EP_8x6mm_P1.27mm_EP3.4x4.3mm -> Package_DFN_QFN:DFN-10-1EP_2.6x2.6mm_P0.5mm_EP1.3x2.2mm
- U4: value BMI270 -> USBLC6-2SC6; footprint footprints:XDCR_BMI270 -> Package_TO_SOT_SMD:SOT-23-6
- U5: value TPS54202DDC -> XC6220B331MR; footprint Package_TO_SOT_SMD:SOT-23-6 -> Package_TO_SOT_SMD:SOT-23-5
- U6: value XC6220B331MR -> STM32F722RETx; footprint Package_TO_SOT_SMD:SOT-23-5 -> Package_QFP:LQFP-64_10x10mm_P0.5mm; moved to B.Cu
- U7: value SPL06-001 -> BMI270; footprint Package_LGA:Bosch_LGA-8_2x2.5mm_P0.65mm_ClockwisePinNumbering -> footprints:XDCR_BMI270
- Y1: footprint Crystal:Crystal_SMD_2012-2Pin_2.0x1.2mm -> Crystal:Resonator_SMD_Murata_CSTxExxV-3Pin_3.0x1.1mm
- moved H1 106.7 mm to (127.5, 61.1)
- moved H2 100.2 mm to (127.5, 37.1)
- moved H3 77.1 mm to (101.5, 61.1)
- moved H4 74.8 mm to (101.5, 37.1)
- moved U5 51.1 mm to (119.7, 37.9), turned to 0 degrees
- moved L1 47.4 mm to (113.7, 37.4)
- moved J1 44.5 mm to (126.5, 49.1), turned to 90 degrees
- moved C18 42.5 mm to (115.8, 41.8), turned to 180 degrees
- moved C14 42.0 mm to (107.5, 43.9), turned to 90 degrees
- moved C13 38.4 mm to (118.1, 53.8), turned to 90 degrees
- moved C19 38.3 mm to (121.3, 46.5), turned to 90 degrees
- moved J2 37.7 mm to (103.0, 49.1)
- moved U2 37.6 mm to (109.3, 37.8), turned to 0 degrees
- moved C2 36.5 mm to (110.4, 35.6), turned to 180 degrees
- moved C17 34.9 mm to (121.2, 52.7)
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Connections:
- C1 pad 1: GND -> VBUS
- C1 pad 2: Net-(U1-PH0) -> GND
- C13 pad 1: VBUS -> +3V3
- C14 pad 1: VBUS -> +3V3
- C15 pad 1: Net-(U5-BOOT) -> +3V3
- C15 pad 2: Net-(U5-SW) -> GND
- C16 pad 1: +5V -> +3V3
- C16 pad 2: Net-(U5-FB) -> GND
- C17 pad 1: +5V -> +3V3
- C18 pad 1: +5V -> +3V3
- C2 pad 1: Net-(U1-PH1) -> Net-(U2-SW)
- C2 pad 2: GND -> Net-(U2-BST)
- C3 pad 1: Net-(U1-VCAP_1) -> +5V
- C4 pad 1: +3V3 -> +5V
- C5 pad 1: +3V3 -> +5V
- C8 pad 1: +3V3 -> Net-(U6-VCAP_1)
- D3 pad 1: +5V -> GND
- J2 pad 3: +5V -> Net-(J2-Pin_3)
- J2 pad 4: GND -> Net-(J2-Pin_4)
- J3 pad 2: +5V -> Net-(J3-Pin_2)
- J3 pad 3: GND -> +5V
- J4 pad 1: Net-(J4-Pin_1) -> +3V3
- J4 pad 2: Net-(J4-Pin_2) -> GND
- J4 pad 3: +5V -> Net-(J4-Pin_3)
- L1 pad 1: Net-(U5-SW) -> Net-(U2-SW)
- R1 pad 1: +3V3 -> /S1
- R1 pad 2: Net-(U1-NRST) -> Net-(J2-Pin_1)
- R10 pad 1: Net-(U5-FB) -> Net-(U6-BOOT0)
- R11 pad 1: /S1 -> +3V3
- R11 pad 2: Net-(J1-Pin_1) -> Net-(U6-NRST)
- R12 pad 1: /S2 -> +3V3
- R12 pad 2: Net-(J1-Pin_2) -> Net-(U9-IO3)
- R13 pad 1: /S3 -> +3V3
- R13 pad 2: Net-(J1-Pin_3) -> Net-(U9-IO2)
- R14 pad 1: /TAIL -> +3V3
- R14 pad 2: Net-(J1-Pin_4) -> /BARO_SCL
- R15 pad 1: /ESC -> +3V3
- R15 pad 2: Net-(J1-Pin_5) -> /BARO_SDA
- R16 pad 1: /RPM -> /UART4_TX
- R16 pad 2: Net-(J1-Pin_6) -> Net-(J3-Pin_1)
- R17 pad 1: /SBUS -> /UART4_RX
- R17 pad 2: Net-(J1-Pin_7) -> Net-(J3-Pin_2)
- R18 pad 1: /UART3_TX -> /LED_GR
- R19 pad 1: /UART4_TX -> /LED_RD
- R19 pad 2: Net-(J2-Pin_1) -> Net-(D3-A)
- R2 pad 1: Net-(U1-BOOT0) -> /S2
- R2 pad 2: GND -> Net-(J2-Pin_2)
- R21 pad 1: /UART6_TX -> /DSM
- R21 pad 2: Net-(J4-Pin_1) -> Net-(J4-Pin_3)
- R3 pad 1: +3V3 -> /S3
- R3 pad 2: /BARO_SCL -> Net-(J2-Pin_3)
- R4 pad 1: +3V3 -> /TAIL
- R4 pad 2: /BARO_SDA -> Net-(J2-Pin_4)
- R5 pad 1: Net-(J5-CC2) -> /ESC
- R5 pad 2: GND -> Net-(J2-Pin_5)
- R6 pad 1: Net-(J5-CC1) -> /RPM
- R6 pad 2: GND -> Net-(J2-Pin_6)
- R7 pad 1: +3V3 -> /SBUS
- R7 pad 2: Net-(U3-IO2) -> Net-(J2-Pin_7)
- R8 pad 1: +3V3 -> Net-(J1-CC2)
- R8 pad 2: Net-(U3-IO3) -> GND
- R9 pad 1: +5V -> Net-(J1-CC1)
- R9 pad 2: Net-(U5-FB) -> GND
- SW1 pad 2: Net-(U1-BOOT0) -> Net-(U6-BOOT0)
- U1 pad 1: +3V3 -> unconnected-(U1-I/O1-Pad1)
- U1 pad 10: /5V_ADC -> (no net)
- U1 pad 11: /Vx_Curr -> GND
- U1 pad 2: unconnected-(U1-PC13-Pad2) -> (no net)
- U1 pad 3: /LED_GR -> /SBUS
- U1 pad 4: /LED_RD -> (no net)
- U1 pad 5: Net-(U1-PH0) -> +5V
- U1 pad 6: Net-(U1-PH1) -> (no net)
- U1 pad 7: Net-(U1-NRST) -> /RPM
- U1 pad 8: /VBAT_ADC -> (no net)
- U1 pad 9: /Vx_ADC -> /ESC
- U2 pad 1: /USB_D- -> +5V
- U2 pad 2: GND -> VBUS
- U2 pad 3: /USB_D+ -> VBUS
- U2 pad 4: /MCU_D+ -> GND
- U2 pad 5: Net-(D3-A) -> Net-(U2-SW)
- U2 pad 6: /MCU_D- -> Net-(U2-BST)
- U3 pad 1: /FLASH_NSS -> /S2
- U3 pad 2: /FLASH_MISO -> (no net)
- U3 pad 3: Net-(U3-IO2) -> /S1
- U3 pad 4: GND -> (no net)
- U3 pad 5: /FLASH_MOSI -> +5V
- U3 pad 6: /FLASH_SCK -> (no net)
- U3 pad 7: Net-(U3-IO3) -> /TAIL
- U3 pad 8: +3V3 -> (no net)
- U3 pad 9: (no net) -> /S3
- U4 pad 1: /BMI_MISO -> /USB_D-
- U4 pad 2: unconnected-(U4-ASDX-Pad2) -> GND
- U4 pad 3: unconnected-(U4-ASCX-Pad3) -> /USB_D+
- U4 pad 4: /BMI_INT -> /MCU_D+
- U4 pad 5: +3V3 -> Net-(D1-A)
- U4 pad 6: GND -> /MCU_D-
- U5 pad 1: GND -> +5V
- U5 pad 2: Net-(U5-SW) -> GND
- U5 pad 3: VBUS -> +5V
- U5 pad 4: Net-(U5-FB) -> unconnected-(U5-NC-Pad4)
- U5 pad 5: unconnected-(U5-EN-Pad5) -> +3V3
- U6 pad 1: +5V -> +3V3
- U6 pad 2: GND -> unconnected-(U6-PC13-Pad2)
- U6 pad 3: +5V -> /LED_GR
- U6 pad 4: unconnected-(U6-NC-Pad4) -> /LED_RD
- U6 pad 5: +3V3 -> Net-(U6-PH0)
- U7 pad 1: GND -> /BMI_MISO
- U7 pad 3: /BARO_SDA -> unconnected-(U7-ASCX-Pad3)
- U7 pad 4: /BARO_SCL -> /BMI_INT
- U7 pad 5: unconnected-(U7-SDO-Pad5) -> +3V3
- U7 pad 6: +3V3 -> GND
- Y1 pad 1: Net-(U1-PH1) -> Net-(U6-PH1)
- Y1 pad 2: Net-(U1-PH0) -> GND
Routing:
- net +5V: track 78.7 -> 10.2 mm, vias 6 -> 7
- net /SWCLK: track 0.00 -> 28.5 mm, vias 0 -> 2
- net /UART4_TX: track 0.00 -> 26.4 mm, vias 0 -> 2
- net /SWDIO: track 0.00 -> 25.9 mm, vias 0 -> 2
- net /UART4_RX: track 0.00 -> 23.7 mm, vias 0 -> 2
- net Net-(U6-BOOT0): track 0.00 -> 22.0 mm, vias 0 -> 2
- net Net-(D1-A): track 0.00 -> 21.4 mm, vias 0 -> 2
- net /S1: track 1.84 -> 21.9 mm, vias 0 -> 3
- net /UART6_TX: track 19.7 -> 0.00 mm, vias 2 -> 0
- net VBUS: track 17.8 -> 0.00 mm, vias 0 -> 4
- net /S2: track 2.55 -> 19.8 mm, vias 0 -> 2
- net /UART6_RX: track 16.7 -> 0.00 mm, vias 2 -> 0
- net /SBUS: track 6.08 -> 22.4 mm, vias 0 -> 2
- net Net-(J4-Pin_2): track 15.6 -> 0.00 mm, vias 2 -> 0
- net /S3: track 1.35 -> 16.3 mm, vias 0 -> 2
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- added copper zone on F.Cu, net +3V3
- added copper zone on In1.Cu, net +3V3
- added copper zone on F.Cu, net +5V
- added copper zone on In1.Cu, net +5V
- added copper zone on In3.Cu, net +5V
- added copper zone on In2.Cu, net GND
- added copper zone on In4.Cu, net GND
- added copper zone on In1.Cu, net VBUS
- removed copper zone on In2.Cu, net +3V3
- removed copper zone on In1.Cu, net GND
- removed copper zone on In2.Cu, net VBUS
Other:
- board size 45 x 25 mm -> 31 x 29 mm
- copper layers 4 -> 6

Commit message: schematic visual updates
Changed lines of the file:
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@@
         (effects (font (size 1 1) (thickness 0.15)))
     )
-    (fp_text value "Outputs" (at -2.54 20.11) (layer "F.Fab")
+    (fp_text value "Outputs" (at 10.1 12.6) (layer "F.Fab")
         (effects (font (size 1 1) (thickness 0.15)))
     )
@@
     (fp_arc (start 2.319501 -1.9055) (mid 3.23874 -1.524738) (end 3.6195 -0.605499)
       (stroke (width 0.2) (type solid)) (layer "F.SilkS"))
-    (fp_arc (start 3.6195 0.605498) (mid 3.238739 1.524738) (end 2.3195 1.9055)
+    (fp_arc (start 3.6195 0.605498) (mid 3.23874 1.524738) (end 2.3195 1.9055)
       (stroke (width 0.2) (type solid)) (layer "F.SilkS"))
     (fp_line (start -1.27 -0.635) (end 1.27 -0.635)
@@
     (polygon
       (pts
-        (xy 95.49 31.13)
-        (xy 134.49 31.13)
-        (xy 134.49 68.13)
-        (xy 95.49 68.13)
+        (xy 96.49 32.13)
+        (xy 132.49 32.13)
+        (xy 132.49 66.13)
+        (xy 96.49 66.13)
       )
     )
@@
     (polygon
       (pts
-        (xy 96.49 32.13)
-        (xy 133.99 32.13)
-        (xy 133.99 67.13)
-        (xy 96.49 67.13)
+        (xy 97.49 33.13)
+        (xy 131.49 33.13)
+        (xy 131.49 65.13)
+        (xy 97.49 65.13)
       )
     )
