File: RotorflightF7.kicad_sch (KiCad schematic)
At the start: 58 parts, among them J1 Outputs, J2 RX, J3 LED, J4 UART, J5 USB_C_Receptacle_USB2.0, SW1 SW_Push, U1 STM32F722RETx, U2 USBLC6-2SC6, U4 BMI270, U5 TPS54202DDC, U6 XC6220B331MR, Y1 8MHz

Commit message: stuff
Parts:
- removed D1: RED, LED_SMD:LED_0603_1608Metric, symbol Device:LED_Small
- removed D2: GRN, LED_SMD:LED_0603_1608Metric, symbol Device:LED_Small
- added C20, C21: 100n, Capacitor_SMD:C_0402_1005Metric, symbol Device:C_Small
- added D5: LED_KBRG, LED_SMD:LED_WS2812B-2020_PLCC4_2.0x2.0mm, symbol Device:LED_KBRG
- added J6: C, Connector_JST:JST_GH_BM04B-GHS-TBT_1x04-1MP_P1.25mm_Vertical, symbol Connector_Generic:Conn_01x04
- added J7: DSM, Connector_JST:JST_GH_BM04B-GHS-TBT_1x04-1MP_P1.25mm_Vertical, symbol Connector_Generic:Conn_01x03
- added R19, R20, R21, R22, R23, R24, R25: 22, Resistor_SMD:R_0402_1005Metric, symbol Device:R_Small
- added R26: 47, Resistor_SMD:R_0402_1005Metric, symbol Device:R_Small
- added R27: 75, Resistor_SMD:R_0402_1005Metric, symbol Device:R_Small
- added U3: W25N01G, Package_SON:WSON-8-1EP_8x6mm_P1.27mm_EP3.4x4.3mm, symbol bmi270:W225N01GVZEIG
- added U7: SPL06-001, Package_LGA:Bosch_LGA-8_2x2.5mm_P0.65mm_ClockwisePinNumbering, symbol bmi270:SPL06-001
- C1, C10, C11, C12, C13, C15, C16, C18, C19, C2, C3, C4, C5, C6, C7, C8, C9: footprint Capacitor_SMD:C_0603_1608Metric -> Capacitor_SMD:C_0402_1005Metric
- J1: symbol Connector_Generic:Conn_01x24 -> Connector_Generic:Conn_01x21
- J2: value RX -> A; footprint Connector_JST:JST_SH_BM04B-SRSS-TB_1x04-1MP_P1.00mm_Vertical -> Connector_JST:JST_GH_BM04B-GHS-TBT_1x04-1MP_P1.25mm_Vertical
- J3: footprint Connector_JST:JST_SH_BM03B-SRSS-TB_1x03-1MP_P1.00mm_Vertical -> Connector_JST:JST_GH_BM03B-GHS-TBT_1x03-1MP_P1.25mm_Vertical
- J4: value UART -> B; footprint Connector_JST:JST_SH_BM04B-SRSS-TB_1x04-1MP_P1.00mm_Vertical -> Connector_JST:JST_GH_BM04B-GHS-TBT_1x04-1MP_P1.25mm_Vertical
- R1, R10, R2, R5, R6, R7, R8, R9: footprint Resistor_SMD:R_0603_1608Metric -> Resistor_SMD:R_0402_1005Metric
- R11, R12, R13, R14, R15, R16, R17: footprint (none) -> Resistor_SMD:R_0402_1005Metric
- R18: value 470 -> 22; footprint (none) -> Resistor_SMD:R_0402_1005Metric
- R3: value 47 -> 10k; footprint Resistor_SMD:R_0603_1608Metric -> Resistor_SMD:R_0402_1005Metric
- R4: value 75 -> 10k; footprint Resistor_SMD:R_0603_1608Metric -> Resistor_SMD:R_0402_1005Metric
- Y1: footprint Crystal:Crystal_SMD_3225-4Pin_3.2x2.5mm -> Crystal:Crystal_SMD_2012-2Pin_2.0x1.2mm
Connections:
- net +3V3: now also R3.1, R4.1, C20.1, C21.1, J7.1 (Pin_1), U3.8 (VCC), U7.6 (VDDIO), U7.8 (VDD)
- net +5V: now also J6.3 (Pin_3); no longer U2.5 (VBUS)
- net GND: now also J1.15 (Pin_15), J1.16 (Pin_16), C20.2, C21.2, D5.1 (K), J6.4 (Pin_4), J7.3 (Pin_3), U3.4 (GND), U7.1 (GND), U7.7 (GND); no longer J1.22 (Pin_22), J1.23 (Pin_23), J1.24 (Pin_24), R3.1, R4.1
- net LEDOUT: now also U1.41 (PA8), R23.1; no longer J3.1 (Pin_1), U1.55 (PB3)
- net MCU_D+: now also U2.4 (I/O2); no longer U2.6 (I/O1)
- net MCU_D-: now also U2.6 (I/O1); no longer U2.4 (I/O2)
- net USB_D+: now also U2.3 (I/O2); no longer U2.1 (I/O1)
- net USB_D-: now also U2.1 (I/O1); no longer U2.3 (I/O2)
- net VBUS: now also J1.8 (Pin_8); no longer J1.15 (Pin_15), J1.16 (Pin_16)
- net at D3.2 (A), J5.A4 (VBUS), J5.A9 (VBUS)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: now also U2.5 (VBUS)
- net at R18.2: now also J6.1 (Pin_1); no longer J1.8 (Pin_8)
- net at R7.2: now also U3.3 (IO2)
- net 5V_ADC: now reaches U1.10 (PC2)
- net Vx_Curr: now reaches U1.11 (PC3)
- net ESC_Curr: now reaches U1.24 (PC4)
- net LED_GR: now reaches U1.3 (PC14)
- net LED_GR: now also R27.1
- net FLASH_NSS: now reaches U1.33 (PB12)
- net FLASH_NSS: now also U3.1 (~{CS})
- net FLASH_SCK: now reaches U1.34 (PB13)
- net FLASH_SCK: now also U3.6 (CLK)
- net FLASH_MISO: now reaches U1.35 (PB14)
- net FLASH_MISO: now also U3.2 (DO(IO1))
- net FLASH_MOSI: now reaches U1.36 (PB15)
- net FLASH_MOSI: now also U3.5 (DI(IO0))
- net UART6_TX: now reaches U1.37 (PC6)
- net UART6_TX: now also R21.1
- net UART6_RX: now reaches U1.38 (PC7)
- net UART6_RX: now also R22.1
- net LED_RD: now reaches U1.4 (PC15)
- net LED_RD: now also R26.1
- net DSM: now reaches U1.43 (PA10)
- net DSM: now also R25.1
- net VBAT_ADC: now reaches U1.8 (PC0)
- net Vx_ADC: now reaches U1.9 (PC1)
- net BARO_SCL: now reaches R3.2
- net BARO_SCL: now also U1.61 (PB8), U7.4 (SCK)
- net BARO_SDA: now reaches R4.2
- net BARO_SDA: now also U1.62 (PB9), U7.3 (SDI)
- net at R8.2: now also U3.7 (IO3)
- net CS_BMI renamed BMI_NSS
- net BMI_NSS: now also U1.20 (PA4); no longer U1.41 (PA8)
- net CS_FLASH: no longer names the net of U1.42 (PA9)
- net INT1_BMI renamed BMI_INT
- net BMI_INT: now also U1.50 (PA15); no longer U1.49 (PA14)
- net INT2_BMI: no longer names the net of U4.9 (INT2)
- net INT2_BMI: no longer U1.50 (PA15)
- net LED_0 renamed SWDIO
- net OCS_BMI: no longer names the net of U4.10 (OSCB)
- net OCS_BMI: no longer U1.20 (PA4)
- removed net Out1: D4.1 (K1), R11.1, U1.25 (PB0)
- net Out2 renamed S2
- net S2: now also U1.57 (PB5); no longer U1.26 (PB1)
- removed net Out3: D4.4 (K3), R13.1, U1.56 (PB4)
- removed net Out4: D4.5 (K4), R14.1, U1.57 (PB5)
- removed net Out5: D4.6 (K5), R15.1, U1.61 (PB8)
- removed net Out6: D4.7 (K6), R16.1, U1.62 (PB9)
- removed net Out7: D4.8 (K7), R17.1, U1.28 (PB10)
- removed net Out8: D4.9 (K8), R18.1, U1.29 (PB11)
- net SPI_MISO renamed BMI_MISO
- net SPI_MOSI renamed BMI_MOSI
- net SPI_SCK renamed BMI_SCK
- net UART1_RX: no longer names the net of J2.2 (Pin_2)
- net UART1_RX: now also R20.2; no longer U1.59 (PB7)
- net UART1_TX: no longer names the net of J2.1 (Pin_1)
- net UART1_TX: now also R19.2; no longer U1.58 (PB6)
- net UART2_RX: no longer names the net of J4.2 (Pin_2)
- net UART2_RX: now also R22.2; no longer U1.17 (PA3)
- net UART2_TX: no longer names the net of J4.1 (Pin_1)
- net UART2_TX: now also R21.2; no longer U1.16 (PA2)
- new net: J7.2 (Pin_2), R25.2
- new net: J6.2 (Pin_2), R24.2
- new net: D5.2 (BA), R27.2
- new net: D5.3 (RA), R26.2
- new net: J3.1 (Pin_1), R23.2
- new net ESC: D4.4 (K3), R15.1, U1.58 (PB6)
- new net RPM: D4.6 (K5), R16.1, U1.16 (PA2)
- new net S1: D4.9 (K8), R11.1, U1.56 (PB4)
- new net S3: D4.8 (K7), R13.1, U1.25 (PB0)
- new net SBUS: D4.5 (K4), R17.1, U1.17 (PA3)
- new net SWCLK: U1.49 (PA14)
- new net TAIL: D4.7 (K6), R14.1, U1.55 (PB3)
- new net UART3_RX: R24.1, U1.29 (PB11)
- new net UART3_TX: R18.1, U1.28 (PB10)
- new net UART4_RX: R20.1
- new net UART4_TX: R19.1
- no-connect marks 30 -> 25
Other:
- moved on the sheet: C11, C12, D4, J3, J4, U4

Commit message: yes
Parts:
- removed C13, C15: 100n, Capacitor_SMD:C_0402_1005Metric, symbol Device:C_Small
- removed C14: 10u, Capacitor_SMD:C_0603_1608Metric, symbol Device:C_Small
- removed C16: 100p, Capacitor_SMD:C_0402_1005Metric, symbol Device:C_Small
- removed C17: 47u, Capacitor_SMD:C_0603_1608Metric, symbol Device:C_Small
- removed C19: 4.7u, Capacitor_SMD:C_0402_1005Metric, symbol Device:C_Small
- removed D4: DT1240A-08LP3810, Package_DFN_QFN:UDFN-9_1.0x3.8mm_P0.5mm, symbol Power_Protection:DT1240A-08LP3810
- removed D5: LED_KBRG, LED_SMD:LED_WS2812B-2020_PLCC4_2.0x2.0mm, symbol Device:LED_KBRG
- removed H1, H2, H3, H4: MountingHole, MountingHole:MountingHole_3.2mm_M3, symbol Mechanical:MountingHole
- removed J2: A, Connector_JST:JST_GH_BM04B-GHS-TBT_1x04-1MP_P1.25mm_Vertical, symbol Connector_Generic:Conn_01x04
- removed J3: LED, Connector_JST:JST_GH_BM03B-GHS-TBT_1x03-1MP_P1.25mm_Vertical, symbol Connector_Generic:Conn_01x03
- removed J6: C, Connector_JST:JST_GH_BM04B-GHS-TBT_1x04-1MP_P1.25mm_Vertical, symbol Connector_Generic:Conn_01x04
- removed J7: DSM, Connector_JST:JST_GH_BM04B-GHS-TBT_1x04-1MP_P1.25mm_Vertical, symbol Connector_Generic:Conn_01x03
- removed R10: 13.7k, Resistor_SMD:R_0402_1005Metric, symbol Device:R_Small
- removed R18, R19, R20, R23, R24, R25: 22, Resistor_SMD:R_0402_1005Metric, symbol Device:R_Small
- removed R9: 100k, Resistor_SMD:R_0402_1005Metric, symbol Device:R_Small
- removed U5: TPS54202DDC, Package_TO_SOT_SMD:SOT-23-6, symbol Regulator_Switching:TPS54202DDC
- added C3, C4: 22u, Capacitor_SMD:C_0603_1608Metric, symbol Device:C_Small
- added C9: 10u, Capacitor_SMD:C_0603_1608Metric, symbol Device:C_Small
- added D2: Green, LED_SMD:LED_0603_1608Metric, symbol Device:LED_Small
- added D3: Red, LED_SMD:LED_0603_1608Metric, symbol Device:LED_Small
- added H1, H2, H3, H4: MountingHole, MountingHole:MountingHole_2.2mm_M2_Pad_Via, symbol Mechanical:MountingHole_Pad
- added J4: DSM, footprints:JST_ZH_B3B-ZR_1x03_P1.50mm_Vertical, symbol Connector_Generic:Conn_01x03
- added J5: JTAG_TC2030, marbastlib_various:CON_TC2030_outlined, symbol marbastlib_various:JTAG_TC2030
- added R21: 22, Resistor_SMD:R_0402_1005Metric, symbol Device:R_Small
- added U1, U3: ESD1014, Package_DFN_QFN:DFN-10-1EP_2.6x2.6mm_P0.5mm_EP1.3x2.2mm, symbol bmi270:ESD1014
- added U2: AP63205WU, Package_TO_SOT_SMD:TSOT-23-6, symbol bmi270:AP63205
- C1: value 30p -> 10u; footprint Capacitor_SMD:C_0402_1005Metric -> Capacitor_SMD:C_0603_1608Metric
- C2: value 30p -> 100n
- C5: renamed from C18; footprint Capacitor_SMD:C_0402_1005Metric -> Capacitor_SMD:C_0603_1608Metric
- J2: renamed from J1; footprint footprints:8xServo -> footprints:7xServo_Vertical
- J3: renamed from J4; value B -> A
- L1: value 10uH -> CSME0418D-4R7M-LRH; footprint Inductor_SMD:L_Sunlord_MWSA0402S -> Inductor_SMD:L_Vishay_IFSC-1515AH_4x4x1.8mm
- R7: renamed from R17; value 470 -> 22r
- Y1: footprint Crystal:Crystal_SMD_2012-2Pin_2.0x1.2mm -> Crystal:Resonator_SMD_Murata_CSTxExxV-3Pin_3.0x1.1mm; symbol Device:Crystal_Small -> Device:Resonator_Small
- renumbered C4 to C10, C5 to C11, C20 to C12, C11 to C13, C6 to C14, C21 to C15, C12 to C16, C7 to C17, C8 to C18, C9 to C19, C10 to C20, C3 to C8, D3 to D1, J5 to J1, R11 to R1, R2 to R10, R1 to R11, R8 to R12, R7 to R13, R3 to R14, R4 to R15, R21 to R16, R22 to R17, R27 to R18, R26 to R19, R12 to R2, R13 to R3, R14 to R4, R15 to R5, R16 to R6, R5 to R8, R6 to R9, U2 to U4, U6 to U5, U1 to U6, U4 to U7, U7 to U8, U3 to U9
Connections:
- net +3V3: now also C9.1, J4.1 (Pin_1), J5.1 (VCC)
- net +5V: now also C3.1, C4.1, U1.5 (VBUS), U2.1 (FB), U3.5 (VBUS)
- net DSM: now also R21.1
- net ESC: now also U1.9 (I/O4)
- net GND: now also C1.2, Y1.2, C3.2, C4.2, C9.2, D2.1 (K), D3.1 (K), H1.1, H2.1, H3.1, H4.1, J4.2 (Pin_2), J5.5 (GND), U1.11 (GND), U2.4 (GND), U3.11 (GND); no longer C1.1, C2.2
- net RPM: now also U1.7 (I/O3)
- net S1: now also U3.3 (I/O2)
- net S2: now also U3.1 (I/O1)
- net S3: now also U3.9 (I/O4)
- net SBUS: now also U1.3 (I/O2)
- net SWCLK: now also J5.4 (SWCLK)
- net SWDIO: now also J5.2 (SWDIO)
- net TAIL: now also U3.7 (I/O3)
- net UART4_RX: now also R17.1, U6.15 (PA1)
- net UART4_TX: now also R16.1, U6.14 (PA0)
- net UART6_RX: no longer R17.1
- net UART6_TX: no longer R16.1
- net VBUS: now also C1.1, U2.2 (EN), U2.3 (IN)
- net at L1.1: now also C2.1, U2.5 (SW)
- net at R18.2: now also D2.2 (A)
- net at R19.2: now also D3.2 (A)
- net at U6.6 (PH1), Y1.1: no longer C2.1
- new net: C2.2, U2.6 (BST)
- new net: U6.5 (PH0), Y1.3
- new net: J4.3 (Pin_3), R21.2
- no-connect marks 25 -> 23
Other:
- note removed: "DCDC"
- note removed: "Decoupling"
- note removed: "Flash"
- note removed: "IMU"
- note removed: "LEDs"
- note removed: "MCU"
- note removed: "Misc"
- note removed: "Outputs"
- note removed: "Pwr_flag"
- note removed: "USB"
- moved on the sheet: C10, C11, C12, C13, C14, C15, C16, C17, C18, C19, C20, C5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

Commit message: schematic visual updates
Other:
- note added: "Connectors"
- note added: "DCDC"
- note added: "MCU"
- note added: "Misc"
- note added: "Sensors and Flash"
- note added: "Servo outputs"
- note added: "USB"
- moved on the sheet: C1, C10, C11, C12, C13, C14, C15, C16, C17, C18, C19, C2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
